File: hw/tivastep.sch (KiCad schematic (older format))
At the start: 25 parts

Commit message: inputs and supply
Parts:
- added C? (x2): CP2, symbol CP2
- added C? (x2): C, symbol C
- added D? (x2): 5V6, symbol ZENER
- added D?: DIODE, symbol DIODE
- added P?: CONN_01X03, symbol CONN_01X03
- added P?: CONN_01X02, symbol CONN_01X02
- added R? (x2): 18, symbol R
- added R? (x2): 470, symbol R
- added R? (x2): 8k2, symbol R
- added U?: 78L05, symbol 78L05
Connections:
- net labels added: SW1, SW2
- wire segments 64 -> 86

Commit message: second axis hw
Parts:
- removed P?: CONN_01X03, symbol CONN_01X03
- added C? (x5): C, symbol C
- added D? (x8): 5V6, symbol ZENER
- added F? (x2): 50mA PTC, symbol FUSE
- added P?: CONN_01X08, symbol CONN_01X08
- added P? (x2): CONN_01X06, symbol CONN_01X06
- added Q? (x3): NPN, symbol NPN
- added R? (x3): 470, symbol R
- added R? (x6): 8k2, symbol R
- added R? (x6): 18, symbol R
Connections:
- net labels added: DIR1, DIR2, ENA1, ENA2, FLT1, FLT2, PUL1, PUL2, SW3, SW4
- net labels removed: DIR, ENA, FLT, PUL
- wire segments 86 -> 159
