File: hw/tivastep.sch (KiCad schematic (older format))
At the start: 76 parts

Commit message: note: remove R9
Other:
- note added: "NOTE: 0Ohm rezistor R9 has to be removed from Tiva C Lauchpad\n(it's connecting PB6 (mAflt) to PD0 (btn1))"
Changed lines of the file:
@@
 Wire Wire Line
 	2100 1400 2300 1400
+Text Notes 7000 6750 0    60   ~ 0
+NOTE: 0Ohm rezistor R9 has to be removed from Tiva C Lauchpad\n(it's connecting PB6 (mAflt) to  PD0 (btn1))
 $EndSCHEMATC
